Commit message: first commit

File: hector_quadrotor_description/urdf/quadrotor_with_cam.urdf.xacro (robot description, xacro)
@@ -9,5 +9,5 @@
     <xacro:include filename="$(find hector_sensors_description)/urdf/generic_camera.urdf.xacro" />
     <xacro:generic_camera name="front_cam" parent="base_link" ros_topic="camera/image" cam_info_topic="camera/camera_info" update_rate="10" res_x="320" res_y="240" image_format="R8G8B8" hfov="90">
-      <origin xyz="0.05 0.0 -0.06" rpy="0 0 0"/>
+      <origin xyz="0.05 0.0 -0.06" rpy="0 1.57 0"/>
     </xacro:generic_camera>
 </robot>

File: hector_quadrotor_description/urdf/quadrotor_with_downward_cam.urdf.xacro (robot description, xacro)
@@ -6,8 +6,8 @@
     <!-- Instantiate quadrotor_base_macro once (has no parameters atm) -->
     <xacro:quadrotor_base_macro />
-    <!-- Downward facing camera -->
+    <!-- Forward facing camera -->
     <xacro:include filename="$(find hector_sensors_description)/urdf/generic_camera.urdf.xacro" />
     <xacro:generic_camera name="downward_cam" parent="base_link" ros_topic="camera/image" cam_info_topic="camera/camera_info" update_rate="10" res_x="640" res_y="480" image_format="R8G8B8" hfov="90">
-      <origin xyz="0.4 0.0 -0.0" rpy="0 ${M_PI/2} 0"/>
+      <origin xyz="0.05 0.0 -0.06" rpy="0 1.57 0"/>
     </xacro:generic_camera>
 </robot>
