Commit message: first commit

File: hector_quadrotor_description/urdf/quadrotor_downward_cam.gazebo.xacro (robot description, xacro)
@@ -3,4 +3,3 @@
     <xacro:include filename="$(find hector_quadrotor_description)/urdf/quadrotor_downward_cam.urdf.xacro" />
     <xacro:include filename="$(find hector_quadrotor_gazebo)/urdf/quadrotor_plugins.gazebo.xacro" />
-    <xacro:quadrotor_plugins />
 </robot>

File: hector_quadrotor_description/urdf/quadrotor_downward_cam.urdf.xacro (robot description, xacro)
@@ -9,5 +9,6 @@
     <xacro:include filename="$(find hector_sensors_description)/urdf/generic_camera.urdf.xacro" />
     <xacro:generic_camera name="downward_cam" parent="base_link" ros_topic="camera/image" cam_info_topic="camera/camera_info" update_rate="10" res_x="640" res_y="480" image_format="R8G8B8" hfov="90">
-      <origin xyz="0.4 0.0 -0.0" rpy="0 ${M_PI/2} 0"/>
+      <!-- <origin xyz="1.4 0.0 -0.0" rpy="0 0 0"/>   -->
+         <origin xyz="1.4 0.0 -0.0" rpy="0 ${M_PI/2} 0"/>
     </xacro:generic_camera>
 </robot>

File: hector_quadrotor_gazebo/urdf/quadrotor_sensors.gazebo.xacro (robot description, xacro)
@@ -11,8 +11,8 @@
             <rpyOffset>0 0 0</rpyOffset> <!-- deprecated -->
             <gaussianNoise>0</gaussianNoise>  <!-- deprecated -->
-            <accelDrift>0.1 0.1 0.1</accelDrift>
-            <accelGaussianNoise>0.35 0.35 0.3</accelGaussianNoise>
-            <rateDrift>0.1 0.1 0.1</rateDrift>
-            <rateGaussianNoise>0.05 0.05 0.015</rateGaussianNoise>
+            <accelDrift>0.01 0.01 0.01</accelDrift>
+            <accelGaussianNoise>0.035 0.035 0.03</accelGaussianNoise>
+            <rateDrift>0.01 0.01 0.01</rateDrift>
+            <rateGaussianNoise>0.005 0.005 0.0015</rateGaussianNoise>
           </plugin>
           <plugin name="quadrotor_baro_sim" filename="libhector_gazebo_ros_baro.so">
@@ -23,6 +23,6 @@
             <altimeterTopicName>altimeter</altimeterTopicName>
             <offset>0</offset>
-            <drift>10.0</drift>
-            <gaussianNoise>0.1</gaussianNoise>
+            <drift>1.0</drift>
+            <gaussianNoise>0.01</gaussianNoise>
           </plugin>
           <plugin name="quadrotor_magnetic_sim" filename="libhector_gazebo_ros_magnetic.so">
@@ -36,5 +36,5 @@
           </plugin>
           <plugin name="quadrotor_gps_sim" filename="libhector_gazebo_ros_gps.so">
-            <updateRate>4.0</updateRate>
+            <updateRate>4</updateRate>
             <bodyName>base_link</bodyName>
             <frameId>$(arg base_link_frame)</frameId>
