Commit message: PC upload

File: hector_quadrotor_description/urdf/quadrotor_downward_cam.urdf.xacro (robot description, xacro)
@@ -10,5 +10,5 @@
     <xacro:generic_camera name="downward_cam" parent="base_link" ros_topic="camera/image" cam_info_topic="camera/camera_info" update_rate="10" res_x="640" res_y="480" image_format="R8G8B8" hfov="90">
       <!-- <origin xyz="1.4 0.0 -0.0" rpy="0 0 0"/>   -->
-         <origin xyz="1.4 0.0 -0.0" rpy="0 ${M_PI/2} 0"/>
+         <origin xyz="0 0.0 -0.09" rpy="0 ${M_PI/2} 0"/>
     </xacro:generic_camera>
 </robot>
